Commit message: Adds labels for auto segmentation

File: vrx_urdf/wamv_gazebo/urdf/components/wamv_camera.xacro (robot description, xacro)
@@ -1,33 +1,34 @@
 <?xml version="1.0"?>
 <robot xmlns:xacro="http://ros.org/wiki/xacro">
-  <xacro:macro name="wamv_camera" params="name x:=0.5 y:=0 z:=1.5 post_z_from:=1.2965 R:=0 P:=0 Y:=0 post_Y:=0 visualize:=False">
+  <xacro:macro name="wamv_camera"
+    params="name x:=0.5 y:=0 z:=1.5 post_z_from:=1.2965 R:=0 P:=0 Y:=0 post_Y:=0 visualize:=False">
     <!-- Define length variables for link positioning -->
-    <xacro:property name="platform_z" value="${post_z_from}"/>
-    <xacro:property name="post_to_post_arm_x" value="0.03"/>
-    <xacro:property name="post_arm_to_camera_x" value="0.02"/>
-    <xacro:property name="post_arm_to_camera_z" value="0.027"/>
+    <xacro:property name="platform_z" value="${post_z_from}" />
+    <xacro:property name="post_to_post_arm_x" value="0.03" />
+    <xacro:property name="post_arm_to_camera_x" value="0.02" />
+    <xacro:property name="post_arm_to_camera_z" value="0.027" />
     <!-- Monocular Camera -->
     <link name="${namespace}/${name}_link">
       <visual>
-        <origin xyz="-0.033 0 0" rpy="0 0 ${pi/2}"/>
-        <geometry>
-          <mesh filename="package://vrx_gazebo/models/mono_camera/mesh/mono_camera.dae"/>
+        <origin xyz="-0.033 0 0" rpy="0 0 ${pi/2}" />
+        <geometry>
+          <mesh filename="package://vrx_gazebo/models/mono_camera/mesh/mono_camera.dae" />
         </geometry>
       </visual>
       <collision name="${name}_lens_collision">
-        <origin xyz="0.018 0 0" rpy="0 ${pi/2} 0"/>
-        <geometry>
-          <cylinder radius="0.015" length="0.042"/>
+        <origin xyz="0.018 0 0" rpy="0 ${pi/2} 0" />
+        <geometry>
+          <cylinder radius="0.015" length="0.042" />
         </geometry>
       </collision>
       <collision name="${name}_box_collision">
-        <origin xyz="-0.0205 0 0" rpy="0 0 0"/>
-        <geometry>
-          <box size="0.036 0.03 0.03"/>
+        <origin xyz="-0.0205 0 0" rpy="0 0 0" />
+        <geometry>
+          <box size="0.036 0.03 0.03" />
         </geometry>
       </collision>
       <!-- Model inertia as box with <size>0.078 0.03 0.03</size> -->
       <inertial>
-        <mass value="0.3"/>
+        <mass value="0.3" />
         <inertia
           ixx="0.0000450"
@@ -36,5 +37,5 @@
           ixy="0"
           ixz="0"
-          iyz="0"/>
+          iyz="0" />
       </inertial>
     </link>
@@ -44,25 +45,25 @@
     </link>
     <!-- Define post length and mass based on desired z position of sensor -->
-    <xacro:property name="post_length" value="${z-platform_z-post_arm_to_camera_z}"/>
-    <xacro:property name="post_mass_per_meter" value="0.9"/>
-    <xacro:property name="post_mass" value="${post_mass_per_meter * post_length}"/>
-    <xacro:property name="post_radius" value="0.0076"/>
+    <xacro:property name="post_length" value="${z-platform_z-post_arm_to_camera_z}" />
+    <xacro:property name="post_mass_per_meter" value="0.9" />
+    <xacro:property name="post_mass" value="${post_mass_per_meter * post_length}" />
+    <xacro:property name="post_radius" value="0.0076" />
     <!-- Sensor post -->
     <link name="${namespace}/${name}_post_link">
       <visual>
         <geometry>
-          <cylinder radius="${post_radius}" length="${post_length}"/>
+          <cylinder radius="${post_radius}" length="${post_length}" />
         </geometry>
         <material name="${name}_post_material">
-          <color rgba="0.0 0.0 0.0 1.0"/>
+          <color rgba="0.0 0.0 0.0 1.0" />
         </material>
       </visual>
       <collision name="${name}_post_collision">
         <geometry>
-          <cylinder radius="${post_radius}" length="${post_length}"/>
+          <cylinder radius="${post_radius}" length="${post_length}" />
         </geometry>
       </collision>
       <inertial>
-        <mass value="${post_mass}"/>
+        <mass value="${post_mass}" />
         <inertia
           ixx="${(post_mass/12) * (3*post_radius*post_radius + post_length*post_length)}"
@@ -71,5 +72,5 @@
           ixy="0"
           ixz="0"
-          iyz="0"/>
+          iyz="0" />
       </inertial>
     </link>
@@ -77,18 +78,18 @@
     <link name="${namespace}/${name}_post_arm_link">
       <visual name="${name}_post_arm_visual">
-        <origin xyz="-0.038 0 -0.003" rpy="${radians(-60)} 0 ${-pi/2}"/>
-        <geometry>
-          <mesh filename="package://vrx_gazebo/models/sensor_post/mesh/sensor_post_arm.dae"/>
+        <origin xyz="-0.038 0 -0.003" rpy="${radians(-60)} 0 ${-pi/2}" />
+        <geometry>
+          <mesh filename="package://vrx_gazebo/models/sensor_post/mesh/sensor_post_arm.dae" />
         </geometry>
       </visual>
       <collision name="${name}_post_arm_collision">
-        <origin xyz="0 0 0" rpy="${radians(-60)-pi/20} 0 ${-pi/2}"/>
-        <geometry>
-          <cylinder radius="0.008" length="0.065"/>
+        <origin xyz="0 0 0" rpy="${radians(-60)-pi/20} 0 ${-pi/2}" />
+        <geometry>
+          <cylinder radius="0.008" length="0.065" />
         </geometry>
       </collision>
       <inertial>
-        <origin xyz="0 0 0" rpy="${radians(-60)-pi/20} 0 ${-pi/2}"/>
-        <mass value="0.1"/>
+        <origin xyz="0 0 0" rpy="${radians(-60)-pi/20} 0 ${-pi/2}" />
+        <mass value="0.1" />
         <inertia
           ixx="0.00003680833"
@@ -97,12 +98,14 @@
           ixy="0"
           ixz="0"
-          iyz="0"/>
+          iyz="0" />
       </inertial>
     </link>
     <!-- Base to sensor post joint -->
-    <xacro:property name="post_z" value="${platform_z+post_length/2}"/>
-    <xacro:property name="post_to_camera_x" value="${post_to_post_arm_x+post_arm_to_camera_x}"/>
+    <xacro:property name="post_z" value="${platform_z+post_length/2}" />
+    <xacro:property name="post_to_camera_x" value="${post_to_post_arm_x+post_arm_to_camera_x}" />
     <joint name="${namespace}/base_to_${name}_post_joint" type="fixed">
-      <origin xyz="${x-(post_to_camera_x)*cos(post_Y)} ${y-(post_to_camera_x)*sin(post_Y)} ${post_z}" rpy="0 0 ${post_Y}" />
+      <origin
+        xyz="${x-(post_to_camera_x)*cos(post_Y)} ${y-(post_to_camera_x)*sin(post_Y)} ${post_z}"
+        rpy="0 0 ${post_Y}" />
       <parent link="${namespace}/base_link" />
       <child link="${namespace}/${name}_post_link" />
@@ -145,7 +148,7 @@
       <sensor type="camera" name="${name}_sensor">
         <update_rate>30.0</update_rate>
-	<xacro:if value="${visualize}">
-	  <visualize>true</visualize>
-	</xacro:if>
+        <xacro:if value="${visualize}">
+          <visualize>true</visualize>
+        </xacro:if>
         <camera name="${name}_camera">
           <horizontal_fov>1.3962634</horizontal_fov>
@@ -168,5 +171,38 @@
           </noise>
         </camera>
-        </sensor>
+      </sensor>
+      <sensor type="segmentation" name="${name}_instance_segmentation">
+        <topic>panoptic</topic>
+        <segmentation_type>instance</segmentation_type>
+        <update_rate>15.0</update_rate>
+        <always_on>1</always_on>
+        <xacro:if value="${visualize}">
+          <visualize>true</visualize>
+        </xacro:if>
+        <camera name="${name}_segment_camera">
+          <segmentation_type>instance</segmentation_type>
+          <horizontal_fov>1.3962634</horizontal_fov>
+          <image>
+            <width>1280</width>
+            <height>720</height>
+            <format>R8G8B8</format>
+          </image>
+          <clip>
+            <near>0.05</near>
+            <far>400</far>
+          </clip>
+          <noise>
+            <type>gaussian</type>
+            <!-- Noise is sampled independently per pixel on each frame.
+                      That pixel's noise value is added to each of its color
+                      channels, which at that point lie in the range [0,1]. -->
+            <mean>0.0</mean>
+            <stddev>0.000</stddev>
+          </noise>
+          <save enabled="true">
+            <path>segmentation_data/${name}_instance_camera</path>
+          </save>
+        </camera>
+      </sensor>
     </gazebo>
   </xacro:macro>
